File: PCB/_autosave-board.kicad_sch (KiCad schematic)
At the start: 161 parts, among them J1 Micro_SD_Card, J10 Conn_01x10, J11 Conn_01x02, J12 Conn_02x04_Odd_Even, J13 Conn_01x02, J14 Conn_01x02, J15 Conn_01x03, J16 Conn_01x02, J17 Conn_01x05, J18 Conn_01x04, J19 Conn_01x04, J2 Conn_ARM_JTAG_SWD_10, J20 Conn_01x02, J21 Conn_01x03, J22 Conn_02x04_Odd_Even, J23 Conn_01x04, J24 Conn_01x04, J25 Conn_01x02, J26 Conn_01x03, J27 Conn_02x04_Odd_Even, J28 Conn_01x04, J29 Conn_01x04, J3 USB_C_Receptacle_USB2.0_14P, J30 Conn_01x02, J31 Conn_01x03, J32 Conn_01x02, J33 Conn_01x02, J34 Conn_01x02, J35 Conn_01x02, J36 Conn_01x02, J37 Conn_01x02, J4 Conn_01x04, J5 Conn_01x04, J6 Conn_01x02, J7 Conn_01x03, J8 Conn_02x04_Odd_Even, J9 Conn_01x10, Q1 IRLML6402, Q2 NMOS, Q3 NMOS, Q4 NMOS, Q5 NMOS, Q6 NMOS, SW1 SW_Push, SW2 SW_Push, U1 STM32H743VITx, U2 AP7361C, U4 TMC Stepstick, U5 TMC Stepstick, U6 TMC Stepstick, U7 TMC Stepstick, U8 AP63203WU, Y2 25 MHz

Commit message: added the organization stuff to the journal
Parts:
- D1: footprint Diode_SMD:D_SMA -> Diode_SMD:D_SOD-123
Changed lines of the file:
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@@
 			)
 		)
-		(property "Footprint" "Diode_SMD:D_SMA"
+		(property "Footprint" "Diode_SMD:D_SOD-123"
 			(at 46.99 31.75 0)
 			(effects
